File: Hardware/Irrigation-Control/irrigationControl.brd (EAGLE design)
At the start: 72.1 x 59.7 mm, 56 parts, among them IC1 LD117AS33TR, Q1 SST201, T1 BC846, T2 BC846, T3 DMN3024LSD, U1 ESP-WROOM-32, U2 INTERFACE-CP2102-GMR(QFN28), U3 MT3608, X1 JST-XH-02-PIN-LONG-PAD, X2 JST-XH-02-PIN-LONG-PAD

Commit message: up
Parts:
- added Q2: SST201, transistor-fet:SOT23
- added Q3: (no value), dp_devices:SOT-23
- added R11: 10k, rc-master-smd:R0603
- added X3, X4: JST-XH-02-PIN-LONG-PAD, Rembrandt Electronics - JST XH Connectors v1-0:JST-XH-02-PACKAGE-LONG-PAD
- added X5: JST-XH-03-PIN-LONG-PAD, Rembrandt Electronics - JST XH Connectors v1-0:JST-XH-03-PACKAGE-LONG-PAD
- moved H2 9.25 mm to (69.8, 74.9)
Connections:
- new net GPIO25: Q3.1, U1.10
- new net GPIO34: U1.6, X5.3
- new net GPIO35: R11.1, U1.7, X4.2
- new net N$9: Q3.3, X3.2
- new net VCC_PMOSFET: Q1.1, Q2.2, R_TP.2, U$9.+
- net GND: now also Q3.2, R11.2, X5.1
- net SOLAR+: now also Q2.3
- net VCC_USB: now also Q2.1; no longer Q1.1, R_TP.2, U$9.+
- net VDD3V3: now also X4.1
- net VOUT: now also X3.1, X5.2
Routing:
- net GND: track 2.36 -> 357.8 mm, vias 0 -> 7
- net VDD3V3: track 0.00 -> 133.2 mm, vias 0 -> 6
- net VOUT: track 0.00 -> 99.2 mm, vias 0 -> 1
- net OUT/B+: track 0.00 -> 83.5 mm, vias 0 -> 3
- net VCC_PMOSFET: track 0.00 -> 80.8 mm, vias 0 -> 2
- net VCC_USB: track 2.36 -> 76.6 mm
- net 3.7V: track 0.00 -> 47.9 mm, vias 0 -> 2
- net GPIO1: track 0.00 -> 45.7 mm
- net GPIO35: track 0.00 -> 45.4 mm, vias 0 -> 3
- net GPIO25: track 0.00 -> 45.2 mm
- net GPIO34: track 0.00 -> 44.0 mm, vias 0 -> 1
- net GPIO3: track 0.00 -> 41.1 mm
- net N$11: track 0.00 -> 37.8 mm
- net ON: track 0.00 -> 35.2 mm
- net EN: track 0.00 -> 34.9 mm
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- added copper zone on layer 1, net GND
- added copper zone on layer 16, net GND
