File: Hardware/Irrigation-Control/irrigationControl.sch (EAGLE design)
At the start: 56 parts, among them IC1 LD117AS33TR, Q1 SST201, T1 BC846, T2 BC846, T3 DMN3024LSD, U1 ESP-WROOM-32, U2 INTERFACE-CP2102-GMR(QFN28), U3 MT3608, X1 JST-XH-02-PIN-LONG-PAD, X2 JST-XH-02-PIN-LONG-PAD

Commit message: up
Parts:
- added Q2: SST201, transistor-fet:SST201
- added Q3: (no value), dp_devices:TRANSISTOR_FET_BS170-SOT-23
- added R11: 10k, rc-master-smd:R_0603
- added X3, X4: JST-XH-02-PIN-LONG-PAD, Rembrandt Electronics - JST XH Connectors v1-0:JST-XH-02-PIN-LONG-PAD
- added X5: JST-XH-03-PIN-LONG-PAD, Rembrandt Electronics - JST XH Connectors v1-0:JST-XH-03-PIN-LONG-PAD
Connections:
- new net GPIO25: Q3.G, U1.IO25
- new net GPIO34: U1.IO34, X5-3.S
- new net GPIO35: R11.1, U1.IO35, X4-2.S
- new net N$9: Q3.D, X3-2.S
- new net VCC_PMOSFET: Q1.D, Q2.S, R_TP.2, U$9.+
- net GND: now also Q3.S, R11.2, X5-1.S
- net SOLAR+: now also Q2.G
- net VCC_USB: now also Q2.D; no longer Q1.D, R_TP.2, U$9.+
- net VDD3V3: now also X4-1.S
- net VOUT: now also X3-1.S, X5-2.S
Other:
- note added: "DC/DC BOOST 5v"
- note added: "Sensor LDR"
- note added: "Sensor Soil Hmidity"
- note added: "Valvula solenoide 5v"
- note removed: "DC/DC BOOST"
- moved on the sheet: S1, X1-1, X1-2, X2-1, X2-2
